File: Shutdown Circuit V1.kicad_sch (KiCad schematic)
At the start: 13 parts, among them J1 CHV+, J2 CHV-, J3 PRE, J4 HV interlocks, K1 Kill switch, K2 ECUSAFE, K3 BMS SAFE, K4 IMD SAFE, K5 Fujitsu_FTR-LYAA005x, K6 Fujitsu_FTR-LYCA005x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

Commit message: Version 2
Parts:
- removed J1: CHV+, symbol Connector:Conn_01x01_Pin
- removed J2: CHV-, symbol Connector:Conn_01x01_Pin
- removed J3: PRE, symbol Connector:Conn_01x01_Pin
- removed K1: Kill switch, Relay_THT:Relay_DPDT_Omron_G5V-2, symbol Relay:G5V-2
- removed K2: ECUSAFE, Relay_THT:Relay_DPDT_Omron_G5V-2, symbol Relay:G5V-2
- removed K3: BMS SAFE, Relay_THT:Relay_DPDT_Omron_G5V-2, symbol Relay:G5V-2
- removed K4: IMD SAFE, Relay_THT:Relay_DPDT_Omron_G5V-2, symbol Relay:G5V-2
- removed K5: Fujitsu_FTR-LYAA005x, Relay_THT:Relay_SPST-NO_Fujitsu_FTR-LYAA005x_FormA_Vertical, symbol Relay:Fujitsu_FTR-LYAA005x
- removed K6, K7: Fujitsu_FTR-LYCA005x, Relay_THT:Relay_SPDT_Fujitsu_FTR-LYCA005x_FormC_Vertical, symbol Relay:Fujitsu_FTR-LYCA005x
- removed SW2: Master switch HV, Button_Switch_SMD:SW_SPST_CK_KMS2xxGP, symbol Switch:CK_KMS2xxG
- removed SW3: Kill button punch, Button_Switch_SMD:SW_SPST_CK_KMS2xxGP, symbol Switch:CK_KMS2xxG
- added K1: BMS SAFE, Relay_THT:Relay_DPDT_Fujitsu_FTR-F1C, symbol Relay:Fujitsu_FTR-F1C
- added K2: IMD SAFE, Relay_THT:Relay_DPDT_Fujitsu_FTR-F1C, symbol Relay:Fujitsu_FTR-F1C
- added K3: ECU SAFE, Relay_THT:Relay_DPDT_Fujitsu_FTR-F1C, symbol Relay:Fujitsu_FTR-F1C
- added K4: Pilot Kill switch relay, Relay_THT:Relay_DPDT_Fujitsu_FTR-F1C, symbol Relay:Fujitsu_FTR-F1C
- added K5: RELAY CHV+, Relay_THT:Relay_DPDT_Fujitsu_FTR-F1C, symbol Relay:Fujitsu_FTR-F1C
- added K6: RELAY CHV-, Relay_THT:Relay_DPDT_Fujitsu_FTR-F1C, symbol Relay:Fujitsu_FTR-F1C
- added K7: RELAY PRECHARGE, Relay_THT:Relay_DPDT_Fujitsu_FTR-F1C, symbol Relay:Fujitsu_FTR-F1C
- added K8: SKIDOO_MAIN-ELECTRICAL, Relay_THT:Relay_SPDT_Fujitsu_FTR-LYCA005x_FormC_Vertical, symbol Relay:Fujitsu_FTR-LYCA005x
- added SW1: MSHV, symbol Switch:SW_Push_Open
Connections:
- net +12V: now also K1.5, K2.5, K3.5, K4.5, K4.7
- net BMS safe signal: now also K1.4
- net ECU safe signal: now also K3.4
- net GND: now also K8.A1
- net IMD safe signal: now also K2.4
- net at J4.1 (Pin_1): now also K3.1
- net at J4.6 (Pin_6): now also K4.2
- new net: K4.3, K8.A2, SW1.1 (A)
- new net: K5.5, K5.7, K6.5, K6.7, K7.5, K7.7, SW1.2 (B)
- new net: K1.1, K2.2
- new net: K2.1, K3.2
- new net BMS_CHARGE-ENABLE: K5.4
- new net BMS_PRECHARGE: K7.4
- new net CHV+ POSITIF: K5.8
- new net CHV- POSITIF: K6.8
- new net CPRECHARGE POSITIF: K7.8
- new net ECU_CHV- READY: K6.4
- new net Kill switch connector+: K4.4
- new net LV Supply: K1.2
- new net TO_ECU_RSD: K4.8
- new net battey side: K8.11
- new net fusebox side: K8.14
Other:
- note added: "BMS ET IMD safe signal sont les sigaux à la sortie des circuits de latch"
- note added: "Brake over travel"
- note added: "CAN WATCHDOG"
- note added: "IN SKIDOO MAIN HARNESS"
- note added: "les pins libres des relais BMS SAFE, IMD SAFE et ECU SAFE sont libre pour pouvoir faire un suivi l'ECU si besoin"
- moved on the sheet: J4

Commit message: Version 3
Parts:
- removed SW1: MSHV, symbol Switch:SW_Push_Open
- added K9: ACCESSORIES-MAIN-RELAY, Relay_THT:Relay_SPDT_Fujitsu_FTR-LYCA005x_FormC_Vertical, symbol Relay:Fujitsu_FTR-LYCA005x
- added LA3: ESOK-1, symbol Device:Lamp
- added LA4: ESOK-2, symbol Device:Lamp
- added SW2: MSHV, symbol Switch:SW_SPST
Connections:
- net LV Supply is gone; now on net LV_SUPPLY: K1.2
- net GND: now also K9.A1, LA3.1 (-), LA4.1 (-)
- net at K4.3, K8.A2: now also K9.A2, SW2.1 (A)
- net at K5.5, K5.7, K6.5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: now also K5.2, K6.2, LA3.2 (+), LA4.2 (+), SW2.2 (B)
- net TO-ECU_CHV-_ACTIVE: now reaches K6.1
- net TO-ECU_CHV+_ACTIVE: now reaches K5.1
- net +12V renamed LV_SUPPLY
- net BMS_CHARGE-ENABLE renamed BMS_CHARGE_ENABLE
- net CHV+ POSITIF renamed CHV+ 
- net CHV- POSITIF renamed CHV-
- net CPRECHARGE POSITIF renamed CPRECHARGE 
- net battey side: no longer names the net of K8.11
- net fusebox side: no longer names the net of K8.14
Other:
- note added: "ESOK LAMPS"
- note added: "RELAI POUR LES ACCESSOIRES COMME FAN ET POMPE"
- note added: "les pins libres des relais BMS SAFE, IMD SAFE et ECU SAFE sont libre pour pouvoir faire un suivi avec l'ECU si besoin"
- note removed: "les pins libres des relais BMS SAFE, IMD SAFE et ECU SAFE sont libre pour pouvoir faire un suivi l'ECU si besoin"
- title: Shutdown Circuit V1 -> Shutdown Circuit
- moved on the sheet: K8
